File: FemtoUSB_r1.0.1/femtoUSB_r1.0.0_TQFP_BREADBOARD.brd (EAGLE design)
At the start: 40.6 x 20.3 mm, 27 parts, among them IC1 ATSAMD21E18A-AU

Commit message: Updating FemtoUSB to r1.0.1 (EXPERIMENTAL)
Parts:
- removed U$38: SPST_SMD, femtoduino:SPST_SMD
- added BOOT_BTN: TACTILE_SWITCH_NO_GND_NO_BOSS, omron_tactile_switch:SIDE_ACT_NO_GND_NO_BOSS
- added C10, C11: 12pF, microbuilder:_0402MP
- added U$40: ABS06-107-32.768KHZ-T, crystals:ABS06-107-32.768KHZ-T
- moved LED2 13.5 mm to (34.5, 11.6)
- moved LED1 13.4 mm to (34.5, 13.1)
- moved IC1 4.21 mm to (22.2, 10.4), turned to 135 degrees
- moved C5 3.98 mm to (7.62, 10.5)
- moved BTN 3.18 mm to (4.65, 6.30)
- moved MICRO_B_USB 3.05 mm to (4.77, 13.0)
- moved C7 1.93 mm to (7.62, 13.6)
- moved C6 1.85 mm to (7.62, 12.1)
- moved LDO_VREG 1.08 mm to (11.2, 12.5)
- moved FB1 1.02 mm to (7.87, 6.99)
- moved C8 0.44 mm to (5.49, 3.68)
- moved C9 0.36 mm to (4.39, 3.68)
- moved L1 0.33 mm to (6.60, 3.68)
Connections:
- net GND: now also BOOT_BTN.1, C10.1, C11.1; no longer U$38.2
- net PA00/X32IN: now also C10.2, U$40.1
- net PA01/X32OUT: now also C11.2, U$40.2
- net PA15/XOUT: now also BOOT_BTN.2; no longer U$38.1
Routing:
- net GND: track 73.7 -> 0.00 mm, vias 9 -> 0
- net 3.3V: track 43.1 -> 0.00 mm, vias 7 -> 0
- net VDDANA: track 30.3 -> 0.00 mm, vias 4 -> 0
- net PA03/VREFA/AIN[1]: track 29.2 -> 0.00 mm, vias 3 -> 0
- net PA15/XOUT: track 27.6 -> 0.00 mm, vias 4 -> 0
- net PA06/AIN[6]: track 25.3 -> 0.00 mm
- net PA08/I2S/SD1/I2C: track 22.8 -> 0.00 mm, vias 1 -> 0
- net PA05/AIN[5]: track 22.4 -> 0.00 mm
- net N$32: track 21.7 -> 0.00 mm
- net PA09/I2S/MCK0/I2C: track 21.2 -> 0.00 mm, vias 1 -> 0
- net PA27: track 20.8 -> 0.00 mm, vias 2 -> 0
- net PA04/AIN[4]: track 20.3 -> 0.00 mm
- net VIN: track 20.2 -> 0.00 mm, vias 2 -> 0
- net RESET: track 19.0 -> 0.00 mm, vias 3 -> 0
- net PA07/AIN[7]/I2S/SD[0]: track 17.4 -> 0.00 mm
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- added copper zone on layer 1, net GND
- added copper zone on layer 16, net GND
- removed copper zone on layer 1, net N$2
- removed copper zone on layer 16, net N$2
Other:
- board text added: "r1.0.4 TQFP"
- board text removed: "r1.0.3 TQFP"
