File: FemtoUSB_r1.0.1/femtoUSB_r1.0.0_TQFP_BREADBOARD.sch (EAGLE design)
At the start: 28 parts, among them IC1 ATSAMD21E18A-AU

Commit message: Updating FemtoUSB to r1.0.1 (EXPERIMENTAL)
Parts:
- removed U$12: 1X6_ROUND, pins_1.27mm_pitch:1X6_ROUND
- removed U$38: SPST_SMD, femtoduino:SPST_SMD
- removed U$6: 1X14_ROUND, pins_1.27mm_pitch:1X14_ROUND
- removed U$7: 1X3_ROUND, pins_1.27mm_pitch:1X3_ROUND
- removed U$9: 1X5_ROUND, pins_1.27mm_pitch:1X5_ROUND
- added BOOT_BTN: TACTILE_SWITCH_NO_GND_NO_BOSS, omron_tactile_switch:TACTILE_SWITCH_NO_GND_NO_BOSS
- added C10, C11: 12pF, microbuilder:CAP_CERAMIC_0402MP
- added PINS_LEFT, PINS_RIGHT: (no value), microbuilder:HEADER-1X15
- added U$40: ABS06-107-32.768KHZ-T, crystals:ABS06-107-32.768KHZ-T
Connections:
- net 3.3V: now also PINS_LEFT.3, PINS_RIGHT.2; no longer U$6.3, U$9.2
- net GND: now also BOOT_BTN.1, C10.P$1, C11.P$1, PINS_LEFT.2, PINS_RIGHT.1; no longer U$38.2, U$6.2, U$9.1
- net PA00/X32IN: now also C10.P$2, PINS_RIGHT.9, U$40.XTALIN; no longer U$7.1
- net PA01/X32OUT: now also C11.P$2, PINS_RIGHT.10, U$40.XTALOUT; no longer U$12.1
- net PA02/AIN[0]: now also PINS_RIGHT.11; no longer U$12.2
- net PA03/VREFA/AIN[1]: now also PINS_RIGHT.12; no longer U$12.3
- net PA04/AIN[4]: now also PINS_RIGHT.13; no longer U$12.4
- net PA05/AIN[5]: now also PINS_RIGHT.14; no longer U$12.5
- net PA06/AIN[6]: now also PINS_RIGHT.15; no longer U$12.6
- net PA07/AIN[7]/I2S/SD[0]: now also PINS_LEFT.14; no longer U$6.14
- net PA08/I2S/SD1/I2C: now also PINS_LEFT.13; no longer U$6.13
- net PA09/I2S/MCK0/I2C: now also PINS_LEFT.12; no longer U$6.12
- net PA10/I2S/SCK0: now also PINS_LEFT.11; no longer U$6.11
- net PA11/I2S/FS0: now also PINS_LEFT.10; no longer U$6.10
- net PA15/XOUT: now also BOOT_BTN.2, PINS_RIGHT.6; no longer U$38.1
- net PA16/SERCOM1/PAD[0]/SPI/I2C: now also PINS_LEFT.9; no longer U$6.9
- net PA17/SERCOM1/PAD[1]/SPI/I2C: now also PINS_LEFT.8; no longer U$6.8
- net PA18/SERCOM1/PAD[2]/SPI: now also PINS_LEFT.7; no longer U$6.7
- net PA19/SERCOM1/PAD[3]/SPI: now also PINS_LEFT.6; no longer U$6.6
- net PA22/I2C: now also PINS_LEFT.5; no longer U$6.5
- net PA23/USB/SOF1KHZ/I2C: now also PINS_LEFT.4; no longer U$6.4
- net PA27: now also PINS_RIGHT.7; no longer U$7.3
- net PA28: now also PINS_RIGHT.8; no longer U$7.2
- net PA30/SWCLK: now also PINS_RIGHT.4; no longer U$9.4
- net PA31/SWDIO: now also PINS_RIGHT.5; no longer U$9.5
- net RESET: now also PINS_RIGHT.3; no longer U$9.3
- net VIN: now also PINS_LEFT.1; no longer U$6.1
