File: FemtoUSB_r1.0.1/femtoUSB_r1.0.0_panelized.sch (EAGLE design)
At the start: 26 parts, among them IC1 ATSAMD21E18A-AU

Commit message: Updating FemtoUSB to r1.0.1 (EXPERIMENTAL)
Parts:
- removed PINS_LEFT, PINS_RIGHT: (no value), microbuilder:HEADER-1X15
- added U$12: 1X6_ROUND, pins_1.27mm_pitch:1X6_ROUND
- added U$6: 1X14_ROUND, pins_1.27mm_pitch:1X14_ROUND
- added U$7: 1X3_ROUND, pins_1.27mm_pitch:1X3_ROUND
- added U$9: 1X5_ROUND, pins_1.27mm_pitch:1X5_ROUND
- C1: DIGIKEY_PART 445-4958-1-ND -> (none)
- IC1: value ATSAMD21E18A-AU -> ATSAMD21E18A-MUT; device atmel-samd21:ATSAMD21E18A-AU -> atmel-samd21:ATSAMD21E18A-MUT; DIGIKEY_PART ATSAMD21E18A-AU-ND -> (none)
- LED1: value RED -> YELLOW
- LED2: value GREEN -> BLUE
- R1: DIGIKEY_PART 541-330JCT-ND -> (none)
Connections:
- net 3.3V: now also U$6.3, U$9.2; no longer PINS_LEFT.3, PINS_RIGHT.2
- net GND: now also U$6.2, U$9.1; no longer PINS_LEFT.2, PINS_RIGHT.1
- net PA00/X32IN: now also U$7.1; no longer PINS_RIGHT.9
- net PA01/X32OUT: now also U$12.1; no longer PINS_RIGHT.10
- net PA02/AIN[0]: now also U$12.2; no longer PINS_RIGHT.11
- net PA03/VREFA/AIN[1]: now also U$12.3; no longer PINS_RIGHT.12
- net PA04/AIN[4]: now also U$12.4; no longer PINS_RIGHT.13
- net PA05/AIN[5]: now also U$12.5; no longer PINS_RIGHT.14
- net PA06/AIN[6]: now also U$12.6; no longer PINS_RIGHT.15
- net PA07/AIN[7]/I2S/SD[0]: now also U$6.14; no longer PINS_LEFT.14
- net PA08/I2S/SD1/I2C: now also U$6.13; no longer PINS_LEFT.13
- net PA09/I2S/MCK0/I2C: now also U$6.12; no longer PINS_LEFT.12
- net PA10/I2S/SCK0: now also U$6.11; no longer PINS_LEFT.11
- net PA11/I2S/FS0: now also U$6.10; no longer PINS_LEFT.10
- net PA15/XOUT: no longer PINS_RIGHT.6
- net PA16/SERCOM1/PAD[0]/SPI/I2C: now also U$6.9; no longer PINS_LEFT.9
- net PA17/SERCOM1/PAD[1]/SPI/I2C: now also U$6.8; no longer PINS_LEFT.8
- net PA18/SERCOM1/PAD[2]/SPI: now also U$6.7; no longer PINS_LEFT.7
- net PA19/SERCOM1/PAD[3]/SPI: now also U$6.6; no longer PINS_LEFT.6
- net PA22/I2C: now also U$6.5; no longer PINS_LEFT.5
- net PA23/USB/SOF1KHZ/I2C: now also U$6.4; no longer PINS_LEFT.4
- net PA27: now also U$7.3; no longer PINS_RIGHT.7
- net PA28: now also U$7.2; no longer PINS_RIGHT.8
- net PA30/SWCLK: now also U$9.4; no longer PINS_RIGHT.4
- net PA31/SWDIO: now also U$9.5; no longer PINS_RIGHT.5
- net RESET: now also U$9.3; no longer PINS_RIGHT.3
- net VIN: now also U$6.1; no longer PINS_LEFT.1
Other:
- moved on the sheet: C8
