File: FemtoUSB_r1.0.1/femtoUSB_r1.0.1.brd (EAGLE design)
At the start: 20.7 x 15.2 mm, 29 parts, among them IC1 ATSAMD21E18A-MUT

Commit message: Updating FemtoUSB to r1.0.1 (EXPERIMENTAL)
Parts:
- removed U$38: SPST_SMD, femtoduino:SPST_SMD
- added C10, C11: 12pF, microbuilder:_0402MP
- added R5: 330, microbuilder:_0402MP
- added R6: 100K, microbuilder:_0402MP
- added U$40: ABS06-107-32.768KHZ-T, crystals:ABS06-107-32.768KHZ-T
- added U$43: TACTILE_SWITCH_NO_GND_NO_BOSS, omron_tactile_switch:SIDE_ACT_NO_GND_NO_BOSS
- moved MICRO_B_USB 2.15 mm to (2.24, 8.08)
- moved LDO_VREG 1.59 mm to (8.73, 11.4)
- moved EPSON_TSX1 1.36 mm to (7.58, 5.76)
- moved FB1 0.82 mm to (5.64, 4.32)
- moved C2 0.17 mm to (12.9, 4.39)
- moved R1 0.13 mm to (4.57, 2.67)
- moved R2 0.13 mm to (6.60, 2.67)
Connections:
- new net N$3: MICRO_B_USB.4, R5.1, R6.1
- net 3.3V: now also R6.2
- net GND: now also C10.1, C11.1, U$43.2; no longer U$38.2
- net PA00/X32IN: now also C10.2, U$40.1
- net PA01/X32OUT: now also C11.2, U$40.2
- net PA15/XOUT: now also U$43.1; no longer U$38.1
- net PA23/USB/SOF1KHZ/I2C: now also R5.2
Routing:
- net PA00/X32IN: track 7.36 -> 17.6 mm, vias 1 -> 3
- net PA01/X32OUT: track 5.44 -> 13.0 mm, vias 1 -> 2
- net PA23/USB/SOF1KHZ/I2C: track 11.1 -> 14.5 mm, vias 1 -> 2
- net N$3: track 0.00 -> 2.45 mm
- net PA15/XOUT: track 21.7 -> 20.1 mm
- net PA27: track 10.9 -> 9.31 mm
- net GND: track 74.7 -> 75.9 mm, vias 8 -> 7
- net N$32: track 19.4 -> 20.5 mm
- net VDDANA: track 23.8 -> 23.2 mm
Other:
- board text added: "femto.io"
- board text added: "r1.0.1"
- board text removed: "BOOT"
- board text removed: "femtoduino.com"
- board text removed: "r1.0.0"
