File: FemtoUSB_r1.0.1/femtoUSB_r1.0.1.sch (EAGLE design)
At the start: 28 parts, among them IC1 ATSAMD21E18A-MUT

Commit message: Updating FemtoUSB to r1.0.1 (EXPERIMENTAL)
Parts:
- removed U$38: SPST_SMD, femtoduino:SPST_SMD
- added C10, C11: 12pF, microbuilder:CAP_CERAMIC_0402MP
- added R5: 330, microbuilder:RESISTOR_0402MP
- added R6: 100K, microbuilder:RESISTOR_0402MP
- added U$40: ABS06-107-32.768KHZ-T, crystals:ABS06-107-32.768KHZ-T
- added U$43: TACTILE_SWITCH_NO_GND_NO_BOSS, omron_tactile_switch:TACTILE_SWITCH_NO_GND_NO_BOSS
Connections:
- new net N$3: MICRO_B_USB.ID, R5.1, R6.1
- net 3.3V: now also R6.2
- net GND: now also C10.P$1, C11.P$1, EPSON_TSX1.GND@1, EPSON_TSX1.GND@2, U$43.2; no longer EPSON_TSX1.GND_2, EPSON_TSX1.GND_4, U$38.2
- net PA00/X32IN: now also C10.P$2, U$40.XTALIN
- net PA01/X32OUT: now also C11.P$2, U$40.XTALOUT
- net PA14/XIN: now also EPSON_TSX1.XIN; no longer EPSON_TSX1.XTALIN
- net PA15/XOUT: now also EPSON_TSX1.XOUT, U$43.1; no longer EPSON_TSX1.XTALOUT, U$38.1
- net PA23/USB/SOF1KHZ/I2C: now also R5.2
Other:
- moved on the sheet: FB1
